File: rockets/slider/kicad/_autosave-slider.sch (KiCad schematic (older format))
At the start: 37 parts, among them J1 I2C Breakout, J2 SPI Breakout, J4 Pyro 1 Terminal, M1 Servo X, M2 Servo Y, Q1 IRF540N, Q2 IRF540N, Q3 IRF540N, SW2 SW_SPDT, U1 LM1086-3.3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

Commit message: loads of pcb shiz
Parts:
- gave numbers to parts that had none: 1
Other:
- note removed: "Internal Pulldown"
Changed lines of the file:
@@
 	1    0    0    -1
 $EndComp
-Text Notes 7500 2850 2    50   ~ 0
-Internal Pulldown
 Wire Notes Line
 	3200 700  4900 700
@@
 ARM
 $Comp
-L Switch:SW_SPDT SW?
+L Switch:SW_SPDT SW1
 U 1 1 609207CF
 P 5100 3750
-F 0 "SW?" H 5200 3450 50  0000 C CNN
+F 0 "SW1" H 5200 3450 50  0000 C CNN
 F 1 "SW_SPDT" H 5100 3550 50  0000 C CNN
 F 2 "" H 5100 3750 50  0001 C CNN
@@
 	4700 3850 4700 3900
 $Comp
-L power:GND #PWR?
+L power:GND #PWR019
 U 1 1 60933106
 P 4700 3900
-F 0 "#PWR?" H 4700 3650 50  0001 C CNN
+F 0 "#PWR019" H 4700 3650 50  0001 C CNN
 F 1 "GND" H 4705 3727 50  0000 C CNN
 F 2 "" H 4700 3900 50  0001 C CNN
